File: nerdqaxe++/nerdqaxe++/pi.kicad_sch (KiCad schematic)
At the start: 23 parts, among them J5 Conn_01x12-Socket, J6 Conn_01x12-Socket, J7 Conn_01x12-Header, J8 Conn_01x12-Header, M1 Fan_4pin, M2 Fan_4pin, U30 T-Display-S3, U32 EMC2302-1, U33 TXU0102-DCU, U37 TMP1075, U38 TMP1075

Commit message: Nerdqaxe++ rev6.1.2PM
1. BM1370 Footprint solder paste revision
2. Added 2R2 resistor in series with bootstrap cap for CSD95472Q5MC
3. 180nH inductors for CSD
4. Vsense closer to ASICs
5. Fiducials
6. Updated top silkscreen
7. Various changes in tracing
Parts:
- U30: Manufacturer (none) -> T-Display S3 [H577]; OrderNr (none) -> T-Display S3 [H577]
Changed lines of the file:
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@@
+			)
+		)
+		(property "Manufacturer" "T-Display S3 [H577]"
+			(at 144.145 64.135 0)
+			(effects
+				(font
+					(size 1.27 1.27)
+				)
+				(hide yes)
+			)
+		)
+		(property "OrderNr" "T-Display S3 [H577]"
+			(at 144.145 64.135 0)
+			(effects
+				(font
+					(size 1.27 1.27)
+				)
+				(hide yes)
 			)
 		)
